Commit message: removed joint_state_publisher

File: urdf/anymal.urdf.xacro (robot description, xacro)
@@ -1423,15 +1423,15 @@
   </hardware>
   <xacro:joint_ros2_control name="LF_HAA" initial_pos="0.0"/>
-  <xacro:joint_ros2_control name="LF_HFE" initial_pos="0.0"/>
-  <xacro:joint_ros2_control name="LF_KFE" initial_pos="0.0"/>
-  <xacro:joint_ros2_control name="RF_HAA" initial_pos="0.0"/>
-  <xacro:joint_ros2_control name="RF_HFE" initial_pos="0.0"/>
-  <xacro:joint_ros2_control name="RF_KFE" initial_pos="0.0"/>
-  <xacro:joint_ros2_control name="LH_HAA" initial_pos="0.0"/>
-  <xacro:joint_ros2_control name="LH_HFE" initial_pos="0.0"/>
-  <xacro:joint_ros2_control name="LH_KFE" initial_pos="0.0"/>
-  <xacro:joint_ros2_control name="RH_HAA" initial_pos="0.0"/>
-  <xacro:joint_ros2_control name="RH_HFE" initial_pos="0.0"/>
-  <xacro:joint_ros2_control name="RH_KFE" initial_pos="0.0"/>
+  <xacro:joint_ros2_control name="LF_HFE" initial_pos="0.03"/>
+  <xacro:joint_ros2_control name="LF_KFE" initial_pos="0.4"/>
+  <xacro:joint_ros2_control name="RF_HAA" initial_pos="-0.8"/>
+  <xacro:joint_ros2_control name="RF_HFE" initial_pos="-0.03"/>
+  <xacro:joint_ros2_control name="RF_KFE" initial_pos="0.4"/>
+  <xacro:joint_ros2_control name="LH_HAA" initial_pos="-0.8"/>
+  <xacro:joint_ros2_control name="LH_HFE" initial_pos="0.03"/>
+  <xacro:joint_ros2_control name="LH_KFE" initial_pos="-0.4"/>
+  <xacro:joint_ros2_control name="RH_HAA" initial_pos="0.8"/>
+  <xacro:joint_ros2_control name="RH_HFE" initial_pos="-0.03"/>
+  <xacro:joint_ros2_control name="RH_KFE" initial_pos="-0.4"/>
 </ros2_control>
 <gazebo reference="lidar">

File: urdf/arm.urdf.xacro (robot description, xacro)
@@ -1,4 +1,7 @@
 <?xml version="1.0"?>
 <robot xmlns:xacro="http://www.ros.org/wiki/xacro" name="arm">
+  <material name="red">
+    <color rgba="1 0 0 1"/>
+  </material>
   <link name="base_link">
     <visual>
@@ -7,4 +10,5 @@
       </geometry>
       <origin rpy="0 0 0" xyz="0 0 0"/>
+      <material name="red"/>
     </visual>
     <collision>
@@ -63,5 +67,5 @@
     <inertial>
       <mass value="0.1"/>
-      <inertia ixx="3.41992001e+06" ixy="0.0" ixz="0.0" iyy="2.85587836e+06" iyz="0.0" izz="5.84313870e+06"/>
+      <inertia ixx="3.41992001" ixy="0.0" ixz="0.0" iyy="2.85587836" iyz="0.0" izz="5.84313870"/>
     </inertial>
   </link>
@@ -86,5 +90,5 @@
      <inertial>
       <mass value="0.1"/>
-      <inertia ixx="6.90013881e+01" ixy="0.0" ixz="0.0" iyy="1.24554875e+02" iyz="0.0" izz="1.04295793e+02"/>
+      <inertia ixx="6.90013881e-03" ixy="0.0" ixz="0.0" iyy="1.24554875e-02" iyz="0.0" izz="1.04295793e-02"/>
     </inertial>
   </link>
@@ -121,5 +125,5 @@
      <inertial>
       <mass value="0.1"/>
-      <inertia ixx="6.90013881e+01" ixy="0.0" ixz="0.0" iyy="1.24554875e+02" iyz="0.0" izz="1.04295793e+02"/>
+      <inertia ixx="6.90013881e-03" ixy="0.0" ixz="0.0" iyy="1.24554875e-02" iyz="0.0" izz="1.04295793e-02"/>
     </inertial>
   </link>
@@ -144,5 +148,5 @@
      <inertial>
       <mass value="0.1"/>
-      <inertia ixx="6.90013881e+01" ixy="0.0" ixz="0.0" iyy="1.24554875e+02" iyz="0.0" izz="1.04295793e+02"/>
+      <inertia ixx="6.90013881e-03" ixy="0.0" ixz="0.0" iyy="1.24554875e-02" iyz="0.0" izz="1.04295793e-02"/>
     </inertial>
   </link>
@@ -154,5 +158,5 @@
     <limit effort="300" velocity="0.1" lower="-3.14" upper="3.14"/>
   </joint>
-  <link name="dyn3_r">
+ <link name="dyn3_r">
   </link>
   <joint name="dyn3_f5" type="fixed">
@@ -179,6 +183,5 @@
     <inertial>
       <mass value="0.1"/>
-      <inertia ixx="1.13130695e+07" ixy="0.0" ixz="0.0" iyy="8.78052401e+06" iyz="0.0" izz="1.72940286e+07"/>
-    </inertial>
+  <inertia ixx="0.001" ixy="0.0" ixz="0.0" iyy="0.001" iyz="0.0" izz="0.001"/>    </inertial>
   </link>
   <joint name="f5_dyn4" type="fixed">
@@ -202,5 +205,5 @@
     <inertial>
       <mass value="0.1"/>
-      <inertia ixx="6.90013881e+01" ixy="0.0" ixz="0.0" iyy="1.24554875e+02" iyz="0.0" izz="1.04295793e+02"/>
+      <inertia ixx="6.90013881e-03" ixy="0.0" ixz="0.0" iyy="1.24554875e-02" iyz="0.0" izz="1.04295793e-02"/>
     </inertial>
   </link>
@@ -237,5 +240,5 @@
      <inertial>
       <mass value="0.1"/>
-      <inertia ixx="6.90013881e+01" ixy="0.0" ixz="0.0" iyy="1.24554875e+02" iyz="0.0" izz="1.04295793e+02"/>
+      <inertia ixx="6.90013881e-03" ixy="0.0" ixz="0.0" iyy="1.24554875e-02" iyz="0.0" izz="1.04295793e-02"/>
     </inertial>
   </link>
@@ -260,5 +263,5 @@
     <inertial>
       <mass value="0.1"/>
-      <inertia ixx="6.90013881e+01" ixy="0.0" ixz="0.0" iyy="1.24554875e+02" iyz="0.0" izz="1.04295793e+02"/>
+      <inertia ixx="6.90013881e-03" ixy="0.0" ixz="0.0" iyy="1.24554875e-02" iyz="0.0" izz="1.04295793e-02"/>
     </inertial>
   </link>
@@ -295,5 +298,5 @@
     <inertial>
       <mass value="0.1"/>
-      <inertia ixx="6.90013881e+01" ixy="0.0" ixz="0.0" iyy="1.24554875e+02" iyz="0.0" izz="1.04295793e+02"/>
+      <inertia ixx="6.90013881e-03" ixy="0.0" ixz="0.0" iyy="1.24554875e-02" iyz="0.0" izz="1.04295793e-02"/>
     </inertial>
   </link>
@@ -321,5 +324,5 @@
     <inertial>
       <mass value="0.1"/>
-      <inertia ixx="6.90013881e+01" ixy="0.0" ixz="0.0" iyy="1.24554875e+02" iyz="0.0" izz="1.04295793e+02"/>
+      <inertia ixx="6.90013881e-03" ixy="0.0" ixz="0.0" iyy="1.24554875e-02" iyz="0.0" izz="1.04295793e-02"/>
     </inertial>
   </link>
@@ -347,5 +350,5 @@
     <inertial>
       <mass value="0.1"/>
-      <inertia ixx="6.90013881e+01" ixy="0.0" ixz="0.0" iyy="1.24554875e+02" iyz="0.0" izz="1.04295793e+02"/>
+      <inertia ixx="6.90013881e-03" ixy="0.0" ixz="0.0" iyy="1.24554875e-02" iyz="0.0" izz="1.04295793e-02"/>
     </inertial>
   </link>
@@ -417,5 +420,5 @@
   <xacro:joint_ros2_control name="j0" initial_pos="0.0"/>
   <xacro:joint_ros2_control name="j1" initial_pos="0.0"/>
-  <xacro:joint_ros2_control name="j2" initial_pos="$(arg pos_j2)"/>
+  <xacro:joint_ros2_control name="j2" initial_pos="2.0"/>
   <xacro:joint_ros2_control name="j3" initial_pos="0.0"/>
 </ros2_control>
