Commit message: need to add camera

File: urdf/arm.urdf.xacro (robot description, xacro)
@@ -1,4 +1,4 @@
 <?xml version="1.0"?>
-<robot name="arm">
+<robot xmlns:xacro="http://www.ros.org/wiki/xacro" name="arm">
   <link name="base_link">
     <visual>
@@ -350,4 +350,17 @@
     </inertial>
   </link>
+  <joint name="camera_joint" type="fixed">
+      <parent link="crawer_base"/>
+      <child link="camera_link"/>
+      <origin xyz="0.0 0 0.00" rpy="0 1.57 0"/>
+  </joint>
+  <link name="camera_link">
+      <visual>
+          <geometry>
+              <box size="0.0000010 0.00000003 0.00000003"/>
+          </geometry>
+          <material name="red"/>
+      </visual>
+  </link>
   <gazebo reference="f4">
     <material>Gazebo/Red</material>
@@ -390,4 +403,22 @@
   </gazebo>
   <gazebo>
+    <plugin filename="ign_ros2_control-system" name="ign_ros2_control::IgnitionROS2ControlPlugin">
+    <parameters>$(find arm_description)/config/pos_controller.yaml</parameters>
+    <controller_manager_prefix_node_name>controller_manager</controller_manager_prefix_node_name>
+    </plugin>
+  </gazebo>
+  <xacro:include filename="$(find arm_description)/urdf/ros2_control/joint_initial_pos.xacro"/>
+  <xacro:arg name="pos_j2" default="2.0"/>
+<!--Install with sudo apt install ros-humble-ign-ros2-control-->
+<ros2_control name="GazeboSystem" type="system">
+  <hardware>
+    <plugin>ign_ros2_control/IgnitionSystem</plugin>
+  </hardware>
+  <xacro:joint_ros2_control name="j0" initial_pos="0.0"/>
+  <xacro:joint_ros2_control name="j1" initial_pos="0.0"/>
+  <xacro:joint_ros2_control name="j2" initial_pos="$(arg pos_j2)"/>
+  <xacro:joint_ros2_control name="j3" initial_pos="0.0"/>
+</ros2_control>
+ <gazebo>
 	  <plugin filename="gz-sim-sensors-system"
 		name="gz::sim::systems::Sensors">

Commit message: camera added

File: urdf/arm.urdf.xacro (robot description, xacro)
@@ -353,5 +353,5 @@
       <parent link="crawer_base"/>
       <child link="camera_link"/>
-      <origin xyz="0.0 0 0.00" rpy="0 1.57 0"/>
+      <origin xyz="0.0 0 0.00" rpy="-1.57 -1.57 0"/>
   </joint>
   <link name="camera_link">
@@ -426,5 +426,5 @@
 	</plugin>
   </gazebo>
-  <gazebo reference="crawer_base">
+  <gazebo reference="camera_link">
   <sensor name="camera" type="camera">
     <camera>

Commit message: finito

File: urdf/arm.urdf.xacro (robot description, xacro)
@@ -67,5 +67,5 @@
     <inertial>
       <mass value="0.1"/>
-      <inertia ixx="3.41992001" ixy="0.0" ixz="0.0" iyy="2.85587836" iyz="0.0" izz="5.84313870"/>
+      <inertia ixx="0.001" ixy="0.0" ixz="0.0" iyy="0.001" iyz="0.0" izz="0.001"/>
     </inertial>
   </link>
@@ -90,5 +90,5 @@
      <inertial>
       <mass value="0.1"/>
-      <inertia ixx="6.90013881e-03" ixy="0.0" ixz="0.0" iyy="1.24554875e-02" iyz="0.0" izz="1.04295793e-02"/>
+      <inertia ixx="6.90013881e-05" ixy="0.0" ixz="0.0" iyy="1.24554875e-04" iyz="0.0" izz="1.04295793e-04"/>
     </inertial>
   </link>
@@ -125,5 +125,5 @@
      <inertial>
       <mass value="0.1"/>
-      <inertia ixx="6.90013881e-03" ixy="0.0" ixz="0.0" iyy="1.24554875e-02" iyz="0.0" izz="1.04295793e-02"/>
+      <inertia ixx="6.90013881e-05" ixy="0.0" ixz="0.0" iyy="1.24554875e-04" iyz="0.0" izz="1.04295793e-04"/>
     </inertial>
   </link>
@@ -148,5 +148,5 @@
      <inertial>
       <mass value="0.1"/>
-      <inertia ixx="6.90013881e-03" ixy="0.0" ixz="0.0" iyy="1.24554875e-02" iyz="0.0" izz="1.04295793e-02"/>
+      <inertia ixx="6.90013881e-05" ixy="0.0" ixz="0.0" iyy="1.24554875e-04" iyz="0.0" izz="1.04295793e-04"/>
     </inertial>
   </link>
@@ -205,5 +205,5 @@
     <inertial>
       <mass value="0.1"/>
-      <inertia ixx="6.90013881e-03" ixy="0.0" ixz="0.0" iyy="1.24554875e-02" iyz="0.0" izz="1.04295793e-02"/>
+      <inertia ixx="6.90013881e-05" ixy="0.0" ixz="0.0" iyy="1.24554875e-04" iyz="0.0" izz="1.04295793e-04"/>
     </inertial>
   </link>
@@ -240,5 +240,5 @@
      <inertial>
       <mass value="0.1"/>
-      <inertia ixx="6.90013881e-03" ixy="0.0" ixz="0.0" iyy="1.24554875e-02" iyz="0.0" izz="1.04295793e-02"/>
+      <inertia ixx="6.90013881e-05" ixy="0.0" ixz="0.0" iyy="1.24554875e-04" iyz="0.0" izz="1.04295793e-04"/>
     </inertial>
   </link>
@@ -263,5 +263,5 @@
     <inertial>
       <mass value="0.1"/>
-      <inertia ixx="6.90013881e-03" ixy="0.0" ixz="0.0" iyy="1.24554875e-02" iyz="0.0" izz="1.04295793e-02"/>
+      <inertia ixx="6.90013881e-05" ixy="0.0" ixz="0.0" iyy="1.24554875e-04" iyz="0.0" izz="1.04295793e-04"/>
     </inertial>
   </link>
@@ -298,5 +298,5 @@
     <inertial>
       <mass value="0.1"/>
-      <inertia ixx="6.90013881e-03" ixy="0.0" ixz="0.0" iyy="1.24554875e-02" iyz="0.0" izz="1.04295793e-02"/>
+      <inertia ixx="6.90013881e-05" ixy="0.0" ixz="0.0" iyy="1.24554875e-04" iyz="0.0" izz="1.04295793e-04"/>
     </inertial>
   </link>
@@ -324,5 +324,5 @@
     <inertial>
       <mass value="0.1"/>
-      <inertia ixx="6.90013881e-03" ixy="0.0" ixz="0.0" iyy="1.24554875e-02" iyz="0.0" izz="1.04295793e-02"/>
+      <inertia ixx="6.90013881e-05" ixy="0.0" ixz="0.0" iyy="1.24554875e-04" iyz="0.0" izz="1.04295793e-04"/>
     </inertial>
   </link>
@@ -350,5 +350,5 @@
     <inertial>
       <mass value="0.1"/>
-      <inertia ixx="6.90013881e-03" ixy="0.0" ixz="0.0" iyy="1.24554875e-02" iyz="0.0" izz="1.04295793e-02"/>
+      <inertia ixx="6.90013881e-05" ixy="0.0" ixz="0.0" iyy="1.24554875e-04" iyz="0.0" izz="1.04295793e-04"/>
     </inertial>
   </link>
@@ -414,5 +414,5 @@
   <xacro:arg name="pos_j2" default="2.0"/>
 <!--Install with sudo apt install ros-humble-ign-ros2-control-->
-<ros2_control name="GazeboSystem" type="system">
+<ros2_control name="IgnitionSystem" type="system">
   <hardware>
     <plugin>ign_ros2_control/IgnitionSystem</plugin>

File: urdf/links.urdf (robot description, URDF)
Before this commit: robot arm, 3 links, 2 joints
Joints:
- joint j0: origin xyz=0 0 0.05 -> xyz=0 0 0.1

File: urdf/ros2_control/joint_initial_pos.xacro (robot description, xacro)
@@ -4,5 +4,4 @@
     <joint name="${name}">
         <command_interface name="position"/>
-        <command_interface name="velocity"/>
         <state_interface name="position">
             <param name="initial_value">${initial_pos}</param>
